Commit message: human skeletal model

File: myobody.urdf (robot description, URDF)
Before this commit: robot myobody, 40 links, 39 joints
Links:
- link calcn_l: geometry collision sphere radius=0.085; visual mesh filename=meshes/l_foot.stl
- link calcn_r: geometry collision sphere radius=0.085; visual mesh filename=meshes/r_foot.stl
- link femur_l: geometry collision cylinder length=0.19 radius=0.067; collision cylinder length=0.2 radius=0.080
- link femur_r: geometry collision cylinder length=0.19 radius=0.067; collision cylinder length=0.2 radius=0.080
- link head: geometry collision sphere radius=0.07; collision sphere radius=0.1
- link humerus_l: geometry collision cylinder length=0.260 radius=0.042; visual mesh filename=meshes/humerus_lv.stl
- link humerus_r: geometry collision cylinder length=0.260 radius=0.042; visual mesh filename=meshes/humerus_rv.stl
- link lumbar: geometry collision cylinder length=0.130 radius=0.110; collision cylinder length=0.154 radius=0.080
- link neck: geometry collision cylinder length=0.08 radius=0.05; visual mesh filename=meshes/hat_cervical.stl
- link patella_l: geometry visual mesh filename=meshes/l_patella.stl
- link patella_r: geometry visual mesh filename=meshes/r_patella.stl
- link pelvis: geometry collision sphere radius=0.110; collision sphere radius=0.110
- link radius_l: geometry visual mesh filename=meshes/radius_lv.stl
- link radius_r: geometry visual mesh filename=meshes/radius_rv.stl
- link sacrum: geometry visual mesh filename=meshes/sacrum.stl
- link talus_l: geometry visual mesh filename=meshes/l_talus.stl
- link talus_r: geometry visual mesh filename=meshes/r_talus.stl
- link thoracic: geometry visual mesh filename=meshes/hat_ribs_scap.stl; visual mesh filename=meshes/hat_thoracic.stl
- link tibia_l: geometry collision cylinder length=0.14 radius=0.056; collision cylinder length=0.21 radius=0.048
- link tibia_r: geometry collision cylinder length=0.14 radius=0.056; collision cylinder length=0.21 radius=0.048
- link toes_l: geometry collision cylinder length=0.085 radius=0.02; visual mesh filename=meshes/l_bofoot.stl
- link toes_r: geometry collision cylinder length=0.085 radius=0.02; visual mesh filename=meshes/r_bofoot.stl
- link ulna_l: geometry collision cylinder length=0.236 radius=0.030; visual mesh filename=meshes/ulna_lv.stl
- link ulna_r: geometry collision cylinder length=0.236 radius=0.030; visual mesh filename=meshes/ulna_rv.stl
